Commit message: fix: restore Touch R1 gripper servo in revised end bracket

File: Browser_SDK/assets/urdf/ld-touch/model.urdf (robot description, URDF)
Before this commit: robot touch_r1_leader_arm_preview, 7 links, 6 joints
Links:
- link link_6: geometry visual mesh filename=meshes/link_6-gripper-servo.stl; visual mesh filename=meshes/link_6-horn.stl

Commit message: Update Touch R1 display to complete V3.2 URDF

File: Browser_SDK/assets/urdf/ld-touch/model.urdf (robot description, URDF)
Before this commit: robot touch_r1_leader_arm_preview, 7 links, 6 joints
Links:
- added link left_finger; visual mesh filename=meshes/left_finger-finger.stl
- added link right_finger; visual mesh filename=meshes/right_finger-finger.stl; visual mesh filename=meshes/right_finger-horn.stl
- link link_6: geometry visual mesh filename=meshes/link_6-horn.stl; visual mesh filename=meshes/link_6-servo.stl
Joints:
- added joint joint_7: type continuous, parent link_6, child right_finger, origin xyz=0.006675 0.0541 0.00235 rpy=0 0 0, axis -0 -1 0
- added joint left_finger_joint: type continuous, parent link_6, child left_finger, origin xyz=-0.015325 0.0541 0.00235 rpy=0 0 0, axis 0 -1 0, mimic joint=joint_7 multiplier=-1.0 offset=0.0
- joint joint_3: axis 1 2.2e-09 0 -> 1 0 0; origin xyz=-9.99997e-05 -0.165625 0 rpy=0 0 0 -> xyz=-0.0001 -0.165625 0 rpy=0 0 0
- joint joint_4: axis 1 2.2e-09 0 -> 1 0 0; origin xyz=0.0003623925 0.165625 0.03875 rpy=0 0 0 -> xyz=0.0003623929 0.165625 0.03875 rpy=0 0 0
- joint joint_5: origin xyz=-0.0002311965 0.048745 0.019343455 rpy=0 0 0 -> xyz=-0.0002311964 0.048745 0.019343455 rpy=0 0 0
- joint joint_6: axis 2.2e-09 -1 0 -> -0 -1 0
